Commit message: Update my_robot.urdf
final visual version

File: examples/description/my_robot.urdf (robot description, URDF)
Before this commit: robot my_robot, 1 links, 0 joints
Links:
- added link base_footprint_link
- added link caster_wheel_link; visual sphere radius=0.05
- added link left_wheel_link; visual cylinder length=0.05 radius=0.1
- added link right_wheel_link; visual cylinder length=0.05 radius=0.1
Joints:
- added joint base_caster_wheel_joint: type fixed, parent base_link, child caster_wheel_link, origin xyz=0.2 0.0 -0.05 rpy=0.0 0.0 0.0
- added joint base_joint: type fixrd, parent base_footprint_link, child base_link, origin xyz=0 0 0.1
- added joint base_left_wheel_joint: type continuous, parent base_link, child left_wheel_link, origin xyz=-0.15 0.225 0.0 rpy=0 0 0, axis 0 1 0
- added joint base_right_wheel_joint: type continuous, parent base_link, child left_wheel_link, origin xyz=-0.15 -0.225 0 rpy=0 0 0, axis 0 1 0

Commit message: Update my_robot.urdf
Fixed typos: links and joints

File: examples/description/my_robot.urdf (robot description, URDF)
Before this commit: robot my_robot, 5 links, 4 joints
Links:
- removed link base_footprint_link
- added link base_footprint
Joints:
- joint base_joint: origin xyz=0 0 0.1 -> xyz=0 0 0.1 rpy=0 0 0; parent base_footprint_link -> base_footprint; type fixrd -> fixed
- joint base_right_wheel_joint: child left_wheel_link -> right_wheel_link
