Commit message: Update my_robot.urdf.xacro
Otimização do código com xacro:macro

File: examples/description/my_robot.urdf.xacro (robot description, xacro)
@@ -20,12 +20,4 @@
     <xacro:property name="wheel_radius" value="0.1" />
     <xacro:property name="wheel_length" value="0.05" />
-    <xacro:macro name="example_macro" params="a b c">
-        <link name="dummy_link">
-            <visual>
-                <geometry>
-                </geometry>
-            </visual>
-        </link>
-    </xacro:macro>
     <link name="base_footprint_link"/>
     <link name="base_link">
@@ -47,13 +39,16 @@
         <origin xyz="0 0 ${wheel_radius}"/>
     </joint>
-    <link name="left_wheel_link">
-        <visual>
-            <geometry>
-                <cylinder radius="${wheel_radius}" length="${wheel_length}"/>
-            </geometry>
-            <origin xyz="0.0 0.0 0.0" rpy="${pi / 2.0} 0.0 0.0"/>
-            <material name="gray"/>
-        </visual>
-    </link>
+    <xacro:macro name="wheel_link" params="prefix">
+        <link name="${prefix}_wheel_link">
+            <visual>
+                <geometry>
+                    <cylinder radius="${wheel_radius}" length="${wheel_length}"/>
+                </geometry>
+                <origin xyz="0.0 0.0 0.0" rpy="${pi / 2.0} 0.0 0.0"/>
+                <material name="gray"/>
+            </visual>
+        </link>
+    </xacro:macro>
+    <xacro:wheel_link prefix="left" />
     <joint name="base_left_wheel_joint" type="continuous">
         <parent link="base_link"/>
@@ -62,13 +57,5 @@
         <axis xyz="0 1 0"/>
     </joint>
-    <link name="right_wheel_link">
-        <visual>
-            <geometry>
-                <cylinder radius="${wheel_radius}" length="${wheel_length}"/>
-            </geometry>
-            <origin xyz="0.0 0.0 0.0" rpy="${pi / 2.0} 0.0 0.0"/>
-            <material name="gray"/>
-        </visual>
-    </link>
+    <xacro:wheel_link prefix="right" />
     <joint name="base_right_wheel_joint" type="continuous">
         <parent link="base_link"/>

Commit message: Update my_robot.urdf.xacro
Fixed typo

File: examples/description/my_robot.urdf.xacro (robot description, xacro)
@@ -17,5 +17,5 @@
     <xacro:property name="base_length" value="0.6" />
     <xacro:property name="base_width" value="0.4" />
-    <xacro:property name="base_heigh" value="0.2" />
+    <xacro:property name="base_height" value="0.2" />
     <xacro:property name="wheel_radius" value="0.1" />
     <xacro:property name="wheel_length" value="0.05" />
@@ -24,5 +24,5 @@
         <visual>
             <geometry>
-                <box size="${base_length} ${base_width} ${base_heigh}"/>
+                <box size="${base_length} ${base_width} ${base_height}"/>
             </geometry>
             <origin xyz="0 0 ${base_height / 2.0}" rpy="0 0 0"/>
