Commit message: Update robot_base.xacro
Fixed typo

File: examples/description/robot_base.xacro (robot description, xacro)
@@ -4,5 +4,5 @@
     <xacro:property name="base_length" value="0.6" />
     <xacro:property name="base_width" value="0.4" />
-    <xacro:property name="base_heigh" value="0.2" />
+    <xacro:property name="base_height" value="0.2" />
     <xacro:property name="wheel_radius" value="0.1" />
     <xacro:property name="wheel_length" value="0.05" />
@@ -11,5 +11,5 @@
         <visual>
             <geometry>
-                <box size="${base_length} ${base_width} ${base_heigh}"/>
+                <box size="${base_length} ${base_width} ${base_height}"/>
             </geometry>
             <origin xyz="0 0 ${base_height / 2.0}" rpy="0 0 0"/>

Commit message: Update robot_base.xacro
Fixed typo

File: examples/description/robot_base.xacro (robot description, xacro)
@@ -17,5 +17,5 @@
         </visual>
     </link>
-    <joint name="base_joint" type="fixrd">
+    <joint name="base_joint" type="fixed">
         <parent link="base_footprint_link"/>
         <child link="base_link"/>
@@ -43,5 +43,5 @@
     <joint name="base_right_wheel_joint" type="continuous">
         <parent link="base_link"/>
-        <child link="left_wheel_link"/>
+        <child link="right_wheel_link"/>
         <origin xyz="${-base_length / 4.0} ${- (base_width + wheel_length) / 2.0} 0" rpy="0 0 0"/>
         <axis xyz="0 1 0"/>

Commit message: Update robot_base.xacro
Fixed link and joint from base_footprint

File: examples/description/robot_base.xacro (robot description, xacro)
@@ -7,5 +7,5 @@
     <xacro:property name="wheel_radius" value="0.1" />
     <xacro:property name="wheel_length" value="0.05" />
-    <link name="base_footprint_link"/>
+    <link name="base_footprint"/>
     <link name="base_link">
         <visual>
@@ -18,5 +18,5 @@
     </link>
     <joint name="base_joint" type="fixed">
-        <parent link="base_footprint_link"/>
+        <parent link="base_footprint"/>
         <child link="base_link"/>
         <origin xyz="0 0 ${wheel_radius}"/>

Commit message: Update robot_base.xacro
Added Inertia and Collision properties

File: examples/description/robot_base.xacro (robot description, xacro)
@@ -16,4 +16,12 @@
             <material name="blue"/>
         </visual>
+        <collision>
+            <geometry>
+                <box size="${base_length} ${base_width} ${base_height}"/>
+            </geometry>
+            <origin xyz="0 0 ${base_height / 2.0}" rpy="0 0 0"/>
+        </collision>
+        <xacro:box_inertia m="5.0" l="${base_length}" w="${base_width}" h="${base_height}"
+                           xyz="0 0 ${base_height / 2.0}" rpy="0 0 0" />
     </link>
     <joint name="base_joint" type="fixed">
@@ -31,4 +39,11 @@
                 <material name="gray"/>
             </visual>
+            <collision>
+                <geometry>
+                    <sphere radius="${wheel_radius}" />
+                </geometry>
+                <origin xyz="0.0 0.0 0.0" rpy="${pi / 2.0} 0.0 0.0"/>
+            </collision>
+            <xacro:cylinder_inertia m="1.0" r="${wheel_radius}" l="${wheel_length}" xyz="0.0 0.0 0.0" rpy="${pi / 2.0} 0.0 0.0" />
         </link>
     </xacro:macro>
@@ -55,4 +70,11 @@
             <material name="green"/>
         </visual>
+        <collision>
+            <geometry>
+                <sphere radius="${wheel_radius / 2.0}"/>
+            </geometry>
+            <origin xyz="0.0 0.0 0.0" rpy="0.0 0.0 0.0"/>
+        </collision>
+        <xacro:sphere_inertia m="0.5" r="${wheel_radius / 2.0}" xyz="0.0 0.0 0.0" rpy="0.0 0.0 0.0" />
     </link>
     <joint name="base_caster_wheel_joint" type="fixed">

Commit message: Update robot_base.xacro
Fixed typo > o_xyz and o_rpy

File: examples/description/robot_base.xacro (robot description, xacro)
@@ -23,5 +23,5 @@
         </collision>
         <xacro:box_inertia m="5.0" l="${base_length}" w="${base_width}" h="${base_height}"
-                           xyz="0 0 ${base_height / 2.0}" rpy="0 0 0" />
+                           o_xyz="0 0 ${base_height / 2.0}" o_rpy="0 0 0" />
     </link>
     <joint name="base_joint" type="fixed">
@@ -45,5 +45,5 @@
                 <origin xyz="0.0 0.0 0.0" rpy="${pi / 2.0} 0.0 0.0"/>
             </collision>
-            <xacro:cylinder_inertia m="1.0" r="${wheel_radius}" l="${wheel_length}" xyz="0.0 0.0 0.0" rpy="${pi / 2.0} 0.0 0.0" />
+            <xacro:cylinder_inertia m="1.0" r="${wheel_radius}" l="${wheel_length}" o_xyz="0.0 0.0 0.0" o_rpy="${pi / 2.0} 0.0 0.0" />
         </link>
     </xacro:macro>
@@ -76,10 +76,10 @@
             <origin xyz="0.0 0.0 0.0" rpy="0.0 0.0 0.0"/>
         </collision>
-        <xacro:sphere_inertia m="0.5" r="${wheel_radius / 2.0}" xyz="0.0 0.0 0.0" rpy="0.0 0.0 0.0" />
+        <xacro:sphere_inertia m="0.5" r="${wheel_radius / 2.0}" o_xyz="0.0 0.0 0.0" o_rpy="0.0 0.0 0.0" />
     </link>
     <joint name="base_caster_wheel_joint" type="fixed">
         <parent link="base_link"/>
         <child link="caster_wheel_link"/>
-        <origin xyz="${-base_length / 3.0} 0.0 ${- wheel_radius / 2.0}" rpy="0.0 0.0 0.0"/>
+        <origin xyz="${base_length / 3.0} 0.0 ${- wheel_radius / 2.0}" rpy="0.0 0.0 0.0"/>
     </joint>
 </robot>
