Commit message: Update cm_properties.xacro
Added Inertial Properties

File: examples/description/cm_properties.xacro (robot description, xacro)
@@ -14,3 +14,29 @@
         <color rgba="0.5 0.5 0.5 1"/>
     </material>
+    <xacro:macro name="box_inertia" params="m l w h o_xyz o_rpy" >
+        <inertial>
+            <origin xyz="${o_xyz}" rpy="${o_rpy}" />
+            <mass value="${m}" />
+            <inertia ixx="${(m/12) * (h*h + l*l)}" ixy="0" ixz="0"
+                     iyy="${(m/12) * (w*w + l*l)}" iyz=""
+                     izz="${(m/12) * (h*h + w*w)}" />
+        </inertial>
+    </xacro:macro>
+    <xacro:macro name="cylinder_inertial" params="m r h o_xyz o_rpy">
+        <inertial>
+            <mass value="${m}" />
+            <origin xyz="${o_xyz}" rpy="${o_rpy}" />
+            <inertia ixx="${(m/12) * (3*r*r + l*l)}" ixy="0" ixz="0"
+                     iyy="${(m/12) * (3*r*r + l*l)}" iyz="0"
+                     izz="${(m/2) * (r*r)}" />
+        </inertial>
+    </xacro:macro>
+    <xacro:macro name="sphere_inertia" params="m r o_xyz o_rpy">
+        <mass value="${m}" />
+        <origin xyz="${o_xyz}" rpy="${o_rpy}" />
+        <inertia ixx="${(2/5) * m*r*r}" ixy="0" ixz="0"
+                     iyy="${(2/5) * m*r*r}" iyz="0"
+                     izz="${(2/5) * m*r*r}" />
+    </xacro:macro>
+    <xacro:macro name="cylinder_collision"></xacro:macro>
 </robot>

Commit message: Update cm_properties.xacro
Fixed cylinder_inertia

File: examples/description/cm_properties.xacro (robot description, xacro)
@@ -23,5 +23,5 @@
         </inertial>
     </xacro:macro>
-    <xacro:macro name="cylinder_inertial" params="m r h o_xyz o_rpy">
+    <xacro:macro name="cylinder_inertia" params="m r l o_xyz o_rpy">
         <inertial>
             <mass value="${m}" />
