Commit message: Update robot_base_gazebo.xacro
Reprogramação: Gazebo Classic

File: examples/my_robot_description/urdf/robot_base_gazebo.xacro (robot description, xacro)
@@ -1,21 +1,30 @@
 <?xml version="1.0"?>
 <robot xmlns:xacro="http://www.ros.org/wiki/xacro">
-    <gazebo reference="caster_wheel_link">
-        <mu1 value="0.1" />
-        <mu2 value="0.1" />
-    </gazebo>
-    <gazebo>
-        <plugin filename="gz-sim-joint-state-publisher-system" name="gz::sim::systems::JointStatePublisher" >
-        </plugin>
-    </gazebo>
-    <gazebo>
-        <plugin filename="gz-sim-diff-drive-system" name="gz::sim::systems::DiffDrive">
-            <left_joint>base_left_wheel_joint</left_joint>
-            <right_joint>base_right_wheel_joint</right_joint>
-            <frame_id>odom</frame_id>
-            <child_frame_id>base_footprint</child_frame_id>
-            <wheel_separation>0.45</wheel_separation>
-            <wheel_radius>0.1</wheel_radius>
-        </plugin>
-    </gazebo>
+   <gazebo reference="base_link">
+        <material>Gazebo/Blue</material>
+   </gazebo>
+   <gazebo reference="right_wheel_link">
+        <material>Gazebo/Grey</material>
+   </gazebo>
+   <gazebo reference="left_wheel_link">
+        <material>Gazebo/Grey</material>
+   </gazebo>
+   <gazebo reference="caster_wheel_link">
+        <material>Gazebo/Grey</material>
+        <mu1 value="0.1"/>
+        <mu2 value="0.1"/>
+   </gazebo>
+   <gazebo name="diff_drive_controller" filename="libgazebo_ros_diff_drive.so">
+        <update_rate>50</update_rate>
+        <left_joint>base_left_joint</left_joint>
+        <right_joint>base_right_joint</right_joint>
+        <wheel_separation>0.45</wheel_separation>
+        <wheel_diameter>0.2</wheel_diameter>
+        <publish_odom>true</publish_odom>
+        <publish_odom_tf>true</publish_odom_tf>
+        <publish_wheel_tf>true</publish_wheel_tf>
+        <odometry_topic>odom</odometry_topic>
+        <odometry_frame>odom</odometry_frame>
+        <robot_base_frame>base_footprint</robot_base_frame>
+   </gazebo>
 </robot>
