Commit message: Update lidar.xacro
Joint position corrected
Visual position corrected

File: examples/my_robot_description/urdf/lidar.xacro (robot description, xacro)
@@ -3,5 +3,5 @@
     <link name="scan_link">
         <visual>
-            <origin xyz="0 0 0" rpy="0 0 0"/>
+            <origin xyz="0 0 0.02" rpy="0 0 0"/>
             <geometry>
                 <cylinder radius="0.1" length="0.06"/>
@@ -13,5 +13,5 @@
         <parent link="base_link"/>
         <child link="scan_link"/>
-        <origin xyz="0 0 0.13" rpy="0 0 0"/>
+        <origin xyz="0 0 0.21" rpy="0 0 0"/>
     </joint>
 </robot>

Commit message: Update lidar.xacro
Added collision and inertia
Added Gazebo plugin

File: examples/my_robot_description/urdf/lidar.xacro (robot description, xacro)
@@ -7,6 +7,12 @@
                 <cylinder radius="0.1" length="0.06"/>
             </geometry>
-            <material name="green" />
+            <material name="black" />
         </visual>
+        <collision>
+            <geometry>
+                <cylinder radius="0.1" length="0.06"/>
+            </geometry>
+        </collision>
+        <xacro:cylinder_inertia m="0.1" r="0.1" l="0.06" o_xyz="0 0 0.02" o_rpy="0 0 0" />
     </link>
     <joint name="base_scan_joint" type="fixed">
@@ -15,3 +21,31 @@
         <origin xyz="0 0 0.21" rpy="0 0 0"/>
     </joint>
+    <gazebo reference="scan_link">
+        <material>Gazebo/Black</material>
+        <sensor name="scan" type="ray">
+            <pose> 0 0 0 0 0 0 </pose>
+            <visualize>false</visualize>
+            <update_rate>10</update_rate>
+            <ray>
+                <scan>
+                    <horizontal>
+                        <samples>360</samples>
+                        <min_angle>-3.14</min_angle>
+                        <max_angle>3.14</max_angle>
+                    </horizontal>
+                </scan>
+                <range>
+                    <min>0.3</min>
+                    <max>12</max>
+                </range>
+            </ray>
+            <plugin name="laser_controller" filename="libgazebo_ros_ray_sensor.so">
+                <ros>
+                    <argument>~/out:=scan</argument>
+                </ros>
+                <output_type>sensor_msgs/LaserScan</output_type>
+                <frame_name>laser_frame</frame_name>
+            </plugin>
+        </sensor>
+    </gazebo>
 </robot>
