Commit message: Update bot.urdf.xacro
Nome do arquivo para "base_link" atualizado para "carenagem.stl"

File: bot_description/urdf/bot.urdf.xacro (robot description, xacro)
@@ -19,5 +19,5 @@
             <origin rpy="0 0 0" xyz="0 0 0"/>
             <geometry>
-                <mesh filename="package://bot_description/meshes/base_link.STL"/>
+                <mesh filename="package://bot_description/meshes/carenagem.STL"/>
             </geometry>
         </visual>
@@ -25,5 +25,5 @@
             <origin rpy="0 0 0" xyz="0 0 0"/>
             <geometry>
-                <mesh filename="package://bot_description/meshes/base_link.STL"/>
+                <mesh filename="package://bot_description/meshes/carenagem.STL"/>
             </geometry>
         </collision>

Commit message: Update bot.urdf.xacro

File: bot_description/urdf/bot.urdf.xacro (robot description, xacro)
@@ -142,18 +142,4 @@
         <origin rpy="0 0 0" xyz="-0.04755 0 -0.0275" />
     </joint>
-    <!-- CAN (experimento prático) -->
-    <!--link name="can_link">
-        <visual>
-            <origin rpy="1.57 0 0" xyz="-0.0325 0.0325 0" />
-            <geometry>
-                <mesh filename="package://bot_description/meshes/can.STL"/>
-            </geometry>
-        </visual>
-    </link>
-    <joint name="can_joint" type="fixed">
-        <parent link="base_link"/>
-        <child link="can_link"/>
-        <origin rpy="0 0 0" xyz="0 0 0.078" />
-    </joint-->
     <link name="imu_link">
         <inertial>

Commit message: Update bot.urdf.xacro
Nome do arquivo da roda

File: bot_description/urdf/bot.urdf.xacro (robot description, xacro)
@@ -46,5 +46,5 @@
             <origin rpy="1.57 0 0" xyz="0 0 0" />
             <geometry>
-                <mesh filename="package://bot_description/meshes/wheel_right_link.STL" />
+                <mesh filename="package://bot_description/meshes/wheel.STL" />
             </geometry>
         </visual>
@@ -73,5 +73,5 @@
             <origin rpy="-1.57 0 0" xyz="0 0 0" />
             <geometry>
-                <mesh filename="package://bot_description/meshes/wheel_left_link.STL" />
+                <mesh filename="package://bot_description/meshes/wheel.STL" />
             </geometry>
         </visual>

Commit message: Update bot.urdf.xacro

File: bot_description/urdf/bot.urdf.xacro (robot description, xacro)
@@ -6,166 +6,5 @@
     <!-- ROS 2 Control -->
     <xacro:include filename="$(find bot_description)/urdf/bot_ros2_control.xacro" />
-    <!-- BASE -->
-    <link name="base_footprint"/>
-    <link name="base_link">
-        <inertial>
-            <origin xyz="0 0 0.04" rpy="0.0 0.25 0.3" />
-            <mass value="8.2573504e-01"/>
-            <inertia ixx="2.2124416e-02" ixy="-1.2294101e-04" ixz="3.4938785e-04"
-               iyy="2.1193702e-02" iyz="-5.0120904e-05"
-               izz="2.0064271e-02" />
-        </inertial>
-        <visual>
-            <origin rpy="0 0 0" xyz="0 0 0"/>
-            <geometry>
-                <mesh filename="package://bot_description/meshes/carenagem.STL"/>
-            </geometry>
-        </visual>
-        <collision>
-            <origin rpy="0 0 0" xyz="0 0 0"/>
-            <geometry>
-                <mesh filename="package://bot_description/meshes/carenagem.STL"/>
-            </geometry>
-        </collision>
-    </link>
-    <joint name="base_joint" type="fixed">
-        <parent link="base_footprint"/>
-        <child link="base_link"/>
-        <origin rpy="0 0 0" xyz="0 0 0.033" />
-    </joint>
-    <!-- WHEELS -->
-    <link name="wheel_right_link">
-        <inertial>
-            <origin xyz="0 -0.014 0" rpy="0 0 0" />
-            <mass value="0.0530086090966721" />
-            <inertia ixx="1.88176298336665E-05" ixy="-4.8444933029987E-10" ixz="1.88163708851143E-08"
-                iyy="3.11510738647764E-05" iyz="-6.93560663069607E-11"
-                izz="1.8801969558182E-05" />
-        </inertial>
-        <visual>
-            <origin rpy="1.57 0 0" xyz="0 0 0" />
-            <geometry>
-                <mesh filename="package://bot_description/meshes/wheel.STL" />
-            </geometry>
-        </visual>
-        <collision>
-            <origin xyz="0 -0.015 0" rpy="1.57 0 0"/>
-            <geometry>
-                <sphere radius="0.033"/>
-            </geometry>
-        </collision>
-    </link>
-    <joint name="wheel_right_joint" type="continuous">
-        <parent link="base_link"/>
-        <child link="wheel_right_link"/>
-        <axis xyz="0 1 0"/>
-        <origin rpy="0 0 0" xyz="0 -0.07 0"/>
-    </joint>
-    <link name="wheel_left_link">
-        <inertial>
-            <origin xyz="0 0.014 0" rpy="0 0 0" />
-            <mass value="0.0530086043217644" />
-            <inertia ixx="1.8792911368909E-05"  ixy="3.31256392204584E-10" ixz="-1.14082001662767E-08"
-               iyy="3.11510738759073E-05" iyz="-3.60499245082192E-10"
-               izz="1.88266886146847E-05" />
-        </inertial>
-        <visual>
-            <origin rpy="-1.57 0 0" xyz="0 0 0" />
-            <geometry>
-                <mesh filename="package://bot_description/meshes/wheel.STL" />
-            </geometry>
-        </visual>
-        <collision>
-            <origin xyz="0 0.015 0" rpy="1.57 0 0"/>
-            <geometry>
-                <sphere radius="0.033"/>
-            </geometry>
-        </collision>
-    </link>
-    <joint name="wheel_left_joint" type="continuous">
-        <parent link="base_link"/>
-        <child link="wheel_left_link"/>
-        <axis xyz="0 1 0"/>
-        <origin rpy="0 0 0" xyz="0 0.07 0"/>
-    </joint>
-    <!-- CASTER -->
-    <link name="caster_front_link">
-        <inertial>
-            <origin xyz="3.89968128948481E-07 2.40073004698083E-07 0.00219173397061506" rpy="0 0 0" />
-            <mass value="1.44379265037903E-06" />
-            <inertia ixx="7.23075276010246E-11" ixy="-6.10956883467859E-16" ixz="2.22849693525031E-15"
-               iyy="3.8713793085917E-11"  iyz="2.93909858781952E-15"
-               izz="1.00967486676306E-10" />
-        </inertial>
-        <visual>
-            <origin rpy="0 0 0" xyz="0 0 0"/>
-            <geometry>
-                <mesh filename="package://bot_description/meshes/caster_front_link.STL"/>
-            </geometry>
-        </visual>
-        <collision>
-            <origin xyz="0 0 0" rpy="0 0 0"/>
-            <geometry>
-                <sphere radius="0.005"/>
-            </geometry>
-        </collision>
-    </link>
-    <joint name="caster_front_joint" type="fixed">
-        <parent link="base_link"/>
-        <child link="caster_front_link"/>
-        <origin rpy="0 0 0" xyz="0.04755 0 -0.0275" />
-    </joint>
-    <link name="caster_rear_link">
-        <inertial>
-            <origin xyz="3.8996812895542E-07 2.40073004698083E-07 0.00219173397061509" rpy="0 0 0" />
-            <mass value="1.44379265037902E-06" />
-            <inertia ixx="7.23075276010246E-11" ixy="-6.10956872363424E-16" ixz="2.22849693527207E-15"
-               iyy="3.87137930859167E-11" iyz="2.939098587861E-15"
-               izz="1.00967486676306E-10" />
-        </inertial>
-        <visual>
-            <origin rpy="0 0 0" xyz="0 0 0"/>
-            <geometry>
-                <mesh filename="package://bot_description/meshes/caster_rear_link.STL"/>
-            </geometry>
-        </visual>
-        <collision>
-            <origin xyz="0 0 0" rpy="0 0 0"/>
-            <geometry>
-                <sphere radius="0.005"/>
-            </geometry>
-        </collision>
-    </link>
-    <joint name="caster_rear_joint" type="fixed">
-        <parent link="base_link"/>
-        <child link="caster_rear_link"/>
-        <origin rpy="0 0 0" xyz="-0.04755 0 -0.0275" />
-    </joint>
-    <link name="imu_link">
-        <inertial>
-            <origin xyz="-0.00552433659106688 0.000168210391520346 0.000514000497342681" rpy="0 0 0" />
-            <mass value="0.000528415362211671" />
-            <inertia ixx="1.46176048428261E-08" ixy="1.40015117949421E-10" ixz="-1.99633872937403E-12"
-               iyy="8.59662482954888E-09" iyz="7.52375112767959E-12"
-               izz="2.30279421279312E-08" />
-        </inertial>
-        <visual>
-            <origin xyz="0 0 0" rpy="0 0 0"/>
-            <geometry>
-                <mesh filename="package://bot_description/meshes/imu_link.STL" />
-            </geometry>
-        </visual>
-        <collision>
-            <origin xyz="0 0 0" rpy="0 0 0"/>
-            <geometry>
-                <mesh filename="package://bot_description/meshes/imu_link.STL" />
-            </geometry>
-        </collision>
-    </link>
-    <joint name="imu_joint" type="fixed">
-        <origin xyz="0 0 0.0698986241758014" rpy="0 0 0" />
-        <parent link="base_link" />
-        <child link="imu_link" />
-        <axis xyz="0 0 0" />
-    </joint>
+    <!-- Include robot assembly file-->
+    <xacro:include filename="$(find bot_description)/urdf/bot_assembly.xacro" />
 </robot>
