Commit message: Update lidar.xacro
Ajuste dos valores para coincidir com o robô real

File: my_robot_description/urdf/lidar.xacro (robot description, xacro)
@@ -5,5 +5,5 @@
             <origin xyz="0 0 0.01" rpy="0 0 0"/>
             <geometry>
-                <cylinder radius="0.1" length="0.06"/>
+                <cylinder radius="0.0278" length="0.0413"/>
             </geometry>
             <material name="black" />
@@ -11,13 +11,13 @@
         <collision>
             <geometry>
-                <cylinder radius="0.1" length="0.06"/>
+                <cylinder radius="0.0278" length="0.0413"/>
             </geometry>
         </collision>
-        <xacro:cylinder_inertia m="0.1" r="0.1" l="0.06" o_xyz="0 0 0.02" o_rpy="0 0 0" />
+        <xacro:cylinder_inertia m="0.1" r="0.0278" l="0.0413" o_xyz="0 0 0.02" o_rpy="0 0 0" />
     </link>
     <joint name="base_scan_joint" type="fixed">
         <parent link="base_link"/>
         <child link="scan_link"/>
-        <origin xyz="0 0 0.22" rpy="0 0 0"/>
+        <origin xyz="0 0 0.11" rpy="0 0 0"/>
     </joint>
     <gazebo reference="scan_link">

Commit message: Update lidar.xacro
LiDAR position actualized (based on the real robot)

File: my_robot_description/urdf/lidar.xacro (robot description, xacro)
@@ -19,5 +19,5 @@
         <parent link="base_link"/>
         <child link="scan_link"/>
-        <origin xyz="0 0 0.11" rpy="0 0 0"/>
+        <origin xyz="0.11 0 0.11" rpy="0 0 0"/>
     </joint>
     <gazebo reference="scan_link">
