Commit message: Update robot_base.xacro
Ajuste dos valores para coincidir com o robô real

File: my_robot_description/urdf/robot_base.xacro (robot description, xacro)
@@ -2,9 +2,9 @@
 <robot xmlns:xacro="http://www.ros.org/wiki/xacro" >
     <!--  Variáveis  -->
-    <xacro:property name="base_length" value="0.5" />
-    <xacro:property name="base_width" value="0.3" />
-    <xacro:property name="base_height" value="0.2" />
-    <xacro:property name="wheel_radius" value="0.075" />
-    <xacro:property name="wheel_length" value="0.05" />
+    <xacro:property name="base_length" value="0.3" />
+    <xacro:property name="base_width" value="0.2" />
+    <xacro:property name="base_height" value="0.15" />
+    <xacro:property name="wheel_radius" value="0.0325" />
+    <xacro:property name="wheel_length" value="0.025" />
     <link name="base_footprint"/>
     <link name="base_link">

Commit message: Update robot_base.xacro
Wheels postition's actualized (based on the real robot)

File: my_robot_description/urdf/robot_base.xacro (robot description, xacro)
@@ -52,5 +52,5 @@
         <parent link="base_link"/>
         <child link="left_wheel_link"/>
-        <origin xyz="${-base_length / 4.0} ${(base_width + wheel_length) / 2.0} 0.0" rpy="0 0 0"/>
+        <origin xyz="${(base_length / 4.0)+0.05} ${(base_width + wheel_length) / 2.0} 0.0" rpy="0 0 0"/>
         <axis xyz="0 1 0"/>
     </joint>
@@ -59,5 +59,5 @@
         <parent link="base_link"/>
         <child link="right_wheel_link"/>
-        <origin xyz="${-base_length / 4.0} ${- (base_width + wheel_length) / 2.0} 0" rpy="0 0 0"/>
+        <origin xyz="${(base_length / 4.0)+0.05} ${- (base_width + wheel_length) / 2.0} 0" rpy="0 0 0"/>
         <axis xyz="0 1 0"/>
     </joint>
@@ -81,5 +81,5 @@
         <parent link="base_link"/>
         <child link="caster_wheel_link"/>
-        <origin xyz="${base_length / 3.0} 0.0 ${- wheel_radius / 2.0}" rpy="0.0 0.0 0.0"/>
+        <origin xyz="${-base_length / 3.0} 0.0 ${- wheel_radius / 2.0}" rpy="0.0 0.0 0.0"/>
     </joint>
 </robot>

Commit message: Update robot_base.xacro

File: my_robot_description/urdf/robot_base.xacro (robot description, xacro)
@@ -4,5 +4,5 @@
     <xacro:property name="base_length" value="0.3" />
     <xacro:property name="base_width" value="0.2" />
-    <xacro:property name="base_height" value="0.15" />
+    <xacro:property name="base_height" value="0.1" />
     <xacro:property name="wheel_radius" value="0.0325" />
     <xacro:property name="wheel_length" value="0.025" />
